File: HB-UNI-SEN-PCB/HB-UNI-SEN-PCB.sch (KiCad schematic (older format))
At the start: 15 parts, among them J0 BATT, J1 I2C_1, J2 I2C_2, J3 A0, J4 A1, J5 A2, J6 A3, J7 PROG, SW1 CONFIG_BUTTON, U1 ArduinoProMini, U2 CC1101

Commit message: Updated to v1.5: - Added raw power input - Moved two resistors and some jumpers - Rerouted some tracks
Parts:
- added JR1: RAW, Connector_PinHeader_2.54mm:PinHeader_1x02_P2.54mm_Vertical, symbol HB-UNI-SEN-PCB-rescue:Conn_01x02-conn
- J0, J5, J6: symbol conn:Conn_01x02 -> HB-UNI-SEN-PCB-rescue:Conn_01x02-conn
- J1, J2, J7: symbol conn:Conn_01x04 -> HB-UNI-SEN-PCB-rescue:Conn_01x04-conn
- J3, J4: symbol conn:Conn_01x03 -> HB-UNI-SEN-PCB-rescue:Conn_01x03-conn
- R2, R3: footprint Resistors_THT:R_Axial_DIN0207_L6.3mm_D2.5mm_P10.16mm_Horizontal -> Resistor_THT:R_Axial_DIN0207_L6.3mm_D2.5mm_P2.54mm_Vertical
- SW1: symbol switches:SW_DIP_x01 -> HB-UNI-SEN-PCB-rescue:SW_DIP_x01-switches
Connections:
- net labels added: +12V
- wire segments 73 -> 77
- no-connect marks 7 -> 6
Changed lines of the file:
@@
 $EndDescr
 $Comp
-L conn:Conn_01x04 J1
+L HB-UNI-SEN-PCB-rescue:Conn_01x04-conn J1
 U 1 1 5ABE0D25
 P 6750 1050
@@
 $EndComp
 $Comp
-L conn:Conn_01x04 J2
+L HB-UNI-SEN-PCB-rescue:Conn_01x04-conn J2
 U 1 1 5ABE0DC1
 P 7350 1050
@@
 $EndComp
 $Comp
-L switches:SW_DIP_x01 SW1
+L HB-UNI-SEN-PCB-rescue:SW_DIP_x01-switches SW1
 U 1 1 5ABE0E28
 P 4050 2500
@@
 $EndComp
 $Comp
-L conn:Conn_01x03 J3
+L HB-UNI-SEN-PCB-rescue:Conn_01x03-conn J3
 U 1 1 5ABE1EB3
 P 7350 2350
@@
 $EndComp
 $Comp
-L conn:Conn_01x03 J4
+L HB-UNI-SEN-PCB-rescue:Conn_01x03-conn J4
 U 1 1 5ABE1F38
 P 7350 3200
@@
 $EndComp
 $Comp
-L conn:Conn_01x02 J5
+L HB-UNI-SEN-PCB-rescue:Conn_01x02-conn J5
 U 1 1 5ABE1F9E
 P 7350 3800
@@
 $EndComp
 $Comp
-L conn:Conn_01x02 J6
+L HB-UNI-SEN-PCB-rescue:Conn_01x02-conn J6
 U 1 1 5ABE2007
 P 7350 4450
@@
 F 0 "R2" V 6980 1950 50  0000 C CNN
 F 1 "10K" V 6900 1950 50  0000 C CNN
-F 2 "Resistors_THT:R_Axial_DIN0207_L6.3mm_D2.5mm_P10.16mm_Horizontal" V 6830 1950 50  0001 C CNN
+F 2 "Resistor_THT:R_Axial_DIN0207_L6.3mm_D2.5mm_P2.54mm_Vertical" V 6830 1950 50  0001 C CNN
 F 3 "" H 6900 1950 50  0001 C CNN
 	1    6900 1950
@@
 F 0 "R3" V 6980 2800 50  0000 C CNN
 F 1 "10K" V 6900 2800 50  0000 C CNN
-F 2 "Resistors_THT:R_Axial_DIN0207_L6.3mm_D2.5mm_P10.16mm_Horizontal" V 6830 2800 50  0001 C CNN
+F 2 "Resistor_THT:R_Axial_DIN0207_L6.3mm_D2.5mm_P2.54mm_Vertical" V 6830 2800 50  0001 C CNN
 F 3 "" H 6900 2800 50  0001 C CNN
 	1    6900 2800
@@
 $EndComp
 $Comp
-L conn:Conn_01x02 J0
+L HB-UNI-SEN-PCB-rescue:Conn_01x02-conn J0
 U 1 1 5ABE2E32
 P 1650 900
@@
 $EndComp
 $Comp
-L conn:Conn_01x04 J7
+L HB-UNI-SEN-PCB-rescue:Conn_01x04-conn J7
 U 1 1 5AC3B268
 P 7350 5300
@@
 Connection ~ 1250 900
 NoConn ~ 2600 2000
-NoConn ~ 1150 2000
 NoConn ~ 2600 2400
 NoConn ~ 2600 2600
@@
 Wire Wire Line
 	1250 900  1450 900
+$Comp
+L HB-UNI-SEN-PCB-rescue:Conn_01x02-conn JR1
+U 1 1 5C6E818A
+P 3200 900
+F 0 "JR1" H 3200 1000 50  0000 C CNN
+F 1 "RAW" H 3200 700 50  0000 C CNN
+F 2 "Connector_PinHeader_2.54mm:PinHeader_1x02_P2.54mm_Vertical" H 3200 900 50  0001 C CNN
+F 3 "" H 3200 900 50  0001 C CNN
+	1    3200 900
+	1    0    0    -1
+$EndComp
+$Comp
+L power:GND #PWR0101
+U 1 1 5C6E826E
+P 2650 1050
+F 0 "#PWR0101" H 2650 800 50  0001 C CNN
+F 1 "GND" H 2650 900 50  0000 C CNN
+F 2 "" H 2650 1050 50  0001 C CNN
+F 3 "" H 2650 1050 50  0001 C CNN
+	1    2650 1050
+	1    0    0    -1
+$EndComp
+$Comp
+L power:+12V #PWR0102
+U 1 1 5C6E82C9
+P 700 2000
+F 0 "#PWR0102" H 700 1850 50  0001 C CNN
+F 1 "+12V" H 715 2173 50  0000 C CNN
+F 2 "" H 700 2000 50  0001 C CNN
+F 3 "" H 700 2000 50  0001 C CNN
+	1    700  2000
+	1    0    0    -1
+$EndComp
+$Comp
+L power:+12V #PWR0103
+U 1 1 5C6E830B
+P 2650 900
+F 0 "#PWR0103" H 2650 750 50  0001 C CNN
+F 1 "+12V" H 2665 1073 50  0000 C CNN
+F 2 "" H 2650 900 50  0001 C CNN
+F 3 "" H 2650 900 50  0001 C CNN
+	1    2650 900
+	1    0    0    -1
+$EndComp
+Wire Wire Line
+	3000 900  2650 900
+Wire Wire Line
+	2650 1000 3000 1000
+Wire Wire Line
+	1150 2000 700  2000
+Wire Wire Line
+	2650 1000 2650 1050
 $EndSCHEMATC

Commit message: Added missing capacitor at CC1101
Parts:
- added C1: 10uF, Capacitor_THT:CP_Radial_D4.0mm_P1.50mm, symbol Device:CP
Connections:
- wire segments 77 -> 79
Changed lines of the file:
@@
 Wire Wire Line
 	2650 1000 2650 1050
+$Comp
+L Device:CP C1
+U 1 1 5C6F3B8E
+P 1200 5650
+F 0 "C1" H 1318 5696 50  0000 L CNN
+F 1 "10uF" H 1318 5605 50  0000 L CNN
+F 2 "Capacitor_THT:CP_Radial_D4.0mm_P1.50mm" H 1238 5500 50  0001 C CNN
+F 3 "~" H 1200 5650 50  0001 C CNN
+	1    1200 5650
+	1    0    0    -1
+$EndComp
+Wire Wire Line
+	1200 5800 1200 5900
+Connection ~ 1200 5900
+Wire Wire Line
+	1200 5500 1200 5350
+Connection ~ 1200 5350
 $EndSCHEMATC
